File: KiCAD/SNES2VGA/SNES2VGA.kicad_pcb (KiCad board)
At the start: 2 copper layers, 30.8 x 23.6 mm, 15 parts, among them J1 3.5mm_vertical, P1 AVMulti_Main, P2 VGA

Commit message: Update PCB
Parts:
- C1, C2, C3: value 100uF -> 100-220uF
Other:
- board text added: "100 - 220uF"
- board text removed: "100uF"

Commit message: KiCAD Project Revision
Parts:
- added C6: 100-220uF, SNES2VGA_Library:Cap_SMD_1206, B.Cu at (152.9, 99.9)
- added JP2: NTSC_SYNC, Jumper:SolderJumper-2_P1.3mm_Open_RoundedPad1.0x1.5mm, F.Cu at (153.1, 102.1)
- JP1: value SolderJumper_3_Open -> LUMA_CVBS_SL
- moved R1 1.94 mm to (147.2, 101.7)
- moved JP1 0.62 mm to (149.4, 103.9)
Connections:
- JP1 pad 2: /HSYNC_VGA -> /PAL_SYNC_BEFORE_CAP
- P1 pad 8: (no net) -> /Chroma_SNES
- P2 pad 11: (no net) -> unconnected-(P2-Pad11)
- P2 pad 14: (no net) -> /VSYNC_VGA
- P2 pad 4: (no net) -> unconnected-(P2-Pad4)
Routing:
- net /PAL_SYNC_BEFORE_CAP: track 0.00 -> 12.4 mm, vias 0 -> 1
- net /Luma_SNES: track 30.6 -> 33.0 mm
- net /Green_SNES: track 9.25 -> 8.22 mm
- net /Audio_L_to_VGA: track 12.9 -> 12.2 mm
- net /HSYNC_VGA: vias 0 -> 2
Other:
- net class Default removed
- net class Track removed
- board text added: "220uF"
- board text added: "FOR PAL - 75 Ohm"
- board text added: "NTSC SYNC"
- board text added: "PAL"
- board text added: "SYNC"
- board text removed: "100 - 220uF"
- board text removed: "PAL 75 Ohm"
